Commit message: feat: Add new files for openarm gripper CAN control

File: src/openarm_static_bimanual_description/urdf/openarm_sb_robot.xacro (robot description, xacro)
@@ -310,4 +310,19 @@
       <axis xyz="0 0 -1"/>
       <limit effort="0.0" lower="${-pi * 11.0 / 36.0}" upper="${pi * 11.0 / 36.0}" velocity="0.0"/>
+    </joint>
+    <!-- ===== CAN Gripper Motor (rev8) ===== -->
+    <link name="${prefix}link_gripper_motor">
+      <inertial>
+        <mass value="0.1"/>
+        <origin xyz="0 0 0" rpy="0 0 0"/>
+        <inertia ixx="0.0001" ixy="0" ixz="0" iyy="0.0001" iyz="0" izz="0.0001"/>
+      </inertial>
+    </link>
+    <joint name="${prefix}rev8" type="revolute">
+      <parent link="${prefix}link8"/>
+      <child link="${prefix}link_gripper_motor"/>
+      <origin xyz="-0.0607602 0 0.00876618" rpy="0 0 0"/>
+      <axis xyz="0 0 1"/>
+      <limit effort="7.0" lower="0.0" upper="1.57" velocity="20.943946"/>
     </joint>
     <!-- 그리퍼를 실제로 구동하고 싶을 때만 prismatic 사용 -->

File: src/openarm_static_bimanual_description/urdf/openarm_static_bimanual.urdf.xacro (robot description, xacro)
@@ -65,9 +65,9 @@
         <param name="disable_torque">${disable_torque_eff}</param>
         <param name="prefix">${left_prefix_eff}</param>
-        <param name="motor_types">DM4340,DM4340,DM4340,DM4340,DM4310,DM4310,DM4310</param>
-        <param name="kp">80,80,20,55,5,5,5</param>
-        <param name="kd">2.75,2.5,0.7,0.4,0.7,0.6,0.5</param>
-        <param name="can_device_ids">0x01,0x02,0x03,0x04,0x05,0x06,0x07</param>
-        <param name="can_master_ids">0x11,0x12,0x13,0x14,0x15,0x16,0x17</param>
+        <param name="motor_types">DM4340,DM4340,DM4340,DM4340,DM4310,DM4310,DM4310,DM4310</param>
+        <param name="kp">80,80,20,55,5,5,5,5</param>
+        <param name="kd">2.75,2.5,0.7,0.4,0.7,0.6,0.5,0.5</param>
+        <param name="can_device_ids">0x01,0x02,0x03,0x04,0x05,0x06,0x07,0x08</param>
+        <param name="can_master_ids">0x11,0x12,0x13,0x14,0x15,0x16,0x17,0x18</param>
       </hardware>
       <!-- 각 조인트 인터페이스 명시 -->
@@ -115,4 +115,12 @@
       </joint>
       <joint name="${left_prefix_eff}rev7">
+        <command_interface name="position"/>
+        <command_interface name="effort"/>
+        <state_interface name="position"/>
+        <state_interface name="velocity"/>
+        <state_interface name="effort"/>
+      </joint>
+      <!-- Gripper joint (CAN motor) -->
+      <joint name="${left_prefix_eff}rev8">
         <command_interface name="position"/>
         <command_interface name="effort"/>
@@ -141,9 +149,9 @@
         <param name="disable_torque">${disable_torque_eff}</param>
         <param name="prefix">${right_prefix_eff}</param>
-        <param name="motor_types">DM4340,DM4340,DM4340,DM4340,DM4310,DM4310,DM4310</param>
-        <param name="kp">80,80,20,55,5,5,5</param>
-        <param name="kd">2.75,2.5,0.7,0.4,0.7,0.6,0.5</param>
-        <param name="can_device_ids">0x21,0x22,0x23,0x24,0x25,0x26,0x27</param>
-        <param name="can_master_ids">0x31,0x32,0x33,0x34,0x35,0x36,0x37</param>
+        <param name="motor_types">DM4340,DM4340,DM4340,DM4340,DM4310,DM4310,DM4310,DM4310</param>
+        <param name="kp">80,80,20,55,5,5,5,5</param>
+        <param name="kd">2.75,2.5,0.7,0.4,0.7,0.6,0.5,0.5</param>
+        <param name="can_device_ids">0x21,0x22,0x23,0x24,0x25,0x26,0x27,0x28</param>
+        <param name="can_master_ids">0x31,0x32,0x33,0x34,0x35,0x36,0x37,0x38</param>
       </hardware>
       <joint name="${right_prefix_eff}rev1">
@@ -190,4 +198,12 @@
       </joint>
       <joint name="${right_prefix_eff}rev7">
+        <command_interface name="position"/>
+        <command_interface name="effort"/>
+        <state_interface name="position"/>
+        <state_interface name="velocity"/>
+        <state_interface name="effort"/>
+      </joint>
+      <!-- Gripper joint (CAN motor) -->
+      <joint name="${right_prefix_eff}rev8">
         <command_interface name="position"/>
         <command_interface name="effort"/>
